File: cots_carrier.kicad_pcb (KiCad board)
At the start: 2 copper layers, 57 x 66 mm, 16 parts, among them J1 XT30PW-F, J2 XT30PW-M, U1 COTS Charger, U2 COTS LM2596 Buck

Commit message: Prod files
Parts:
- moved D1 42.5 mm to (180.3, 100.8)
- moved R1 42.5 mm to (180.3, 103.8)
- moved D2 34.9 mm to (153.5, 53.5), turned to 0 degrees
- moved R2 31.2 mm to (156.5, 53.5), turned to 0 degrees
- moved U1 24.4 mm to (149.8, 97.1)
- moved J1 21.3 mm to (153.0, 101.9)
- moved U2 19.2 mm to (171.6, 52.1)
- moved J2 18.9 mm to (171.4, 109.8)
- moved G*** 1.74 mm to (137.7, 104.7)
Routing:
- net Net-(U1-IN+): track 50.7 -> 11.1 mm, vias 0 -> 2
- net Net-(J2-+): track 21.0 -> 23.7 mm, vias 0 -> 1
- net Net-(J1-+): track 8.78 -> 9.44 mm, vias 0 -> 1
- net GND: vias 73 -> 67
Other:
- board text removed: "BATT OUT"
- board text removed: "BUS IN"

Commit message: aircraft carrier silk screen
Parts:
- added G***: LOGO, LOGO, B.Cu at (161.9, 93.7)
- moved G*** 20.6 mm to (170.9, 77.7)
- moved G*** 11.5 mm to (150.0, 77.5)
Routing:
- net Net-(J2-+): track 23.7 -> 24.9 mm
- net Net-(J1-+): track 9.44 -> 8.44 mm
- net Net-(U1-IN+): track 11.1 -> 11.6 mm
